File: Prototype PCBs/Shield v.2/Input Matrix.sch (KiCad schematic (older format))
At the start: 82 parts, among them J1 JumpSwitch, J2 JumpSwitch, J3 JumpSwitch, J4 JumpSwitch, J5 JumpSwitch, J6 JumpSwitch, J7 JumpSwitch, J8 JumpSwitch, SW1 SW_Push, SW10 SW_Push, SW2 SW_Push, SW3 SW_Push, SW4 SW_Push, SW5 SW_Push, SW6 SW_Push, SW7 SW_Push, SW8 SW_Push, SW9 SW_Push

Commit message: V2 Panels. Matrix Input Test Sketch
Parts:
- removed J1, J8: JumpSwitch, Connector_PinHeader_2.54mm:PinHeader_2x08_P2.54mm_Vertical, symbol Custom:JumpSwitch
- added J19B1, J19C1, J19C2, J19D1, J19F1, J19F2, J19G1, J19H1, J26A1, J26B1, J26C1, J26D1, J26E1, J26F1, J26G1, J26H1: Jumper_NO_Small, Connector_PinHeader_2.54mm:PinHeader_1x02_P2.54mm_Vertical, symbol Device:Jumper_NO_Small
- J20: renamed from J2; symbol Custom:JumpSwitch -> Shield-v.2-rescue:JumpSwitch-Custom
- J21: renamed from J3; symbol Custom:JumpSwitch -> Shield-v.2-rescue:JumpSwitch-Custom
- J22: renamed from J4; symbol Custom:JumpSwitch -> Shield-v.2-rescue:JumpSwitch-Custom
- J23: renamed from J5; symbol Custom:JumpSwitch -> Shield-v.2-rescue:JumpSwitch-Custom
- J24: renamed from J6; symbol Custom:JumpSwitch -> Shield-v.2-rescue:JumpSwitch-Custom
- J25: renamed from J7; symbol Custom:JumpSwitch -> Shield-v.2-rescue:JumpSwitch-Custom
- SW1, SW10, SW2, SW3, SW4, SW5, SW6, SW7, SW8, SW9: footprint Button_Switch_SMD:SW_SPST_B3S-1000 -> Kicad Parts:SW_PUSH-12mm_widepinholes
- renumbered D1 to D17, D2 to D18, D3 to D19, D4 to D20, D5 to D21, D6 to D22, D7 to D23, D8 to D24, D9 to D25, D10 to D26, D11 to D27, D12 to D28, D13 to D29, D14 to D30, D15 to D31, D16 to D32, D17 to D33, D18 to D34, D19 to D35, D20 to D36, D21 to D37, D22 to D38, D23 to D39, D24 to D40, D25 to D41, D26 to D42, D27 to D43, D28 to D44, D29 to D45, D30 to D46, D31 to D47, D32 to D48, D33 to D49, D34 to D50, D35 to D51, D36 to D52, D37 to D53, D38 to D54, D39 to D55, D40 to D56, D41 to D57, D42 to D58, D43 to D59, D44 to D60, D45 to D61, D46 to D62, D47 to D63, D48 to D64, D49 to D65, D50 to D66, D51 to D67, D52 to D68, D53 to D69, D54 to D70, D55 to D71, D56 to D72, D57 to D73, D58 to D74, D59 to D75, D60 to D76, D61 to D77, D62 to D78, D63 to D79, D64 to D80
Connections:
- net input_c0: now also D19.2 (A), D20.2 (A), D21.2 (A)
- net input_r0: now also J19C2.1, J26A1.1
- net input_r1: now also J19B1.1, J26B1.1
- net input_r2: now also J19C1.1, J26C1.1
- net input_r3: now also J19D1.1, J26D1.1
- net input_r4: now also J19F1.1, J26E1.1
- net input_r5: now also J19F2.1, J26F1.1
- net input_r6: now also J19G1.1, J26G1.1
- net input_r7: now also J19H1.1, J26H1.1
- net at D77.1 (K), SW10.2: now also J26E1.2
- net at D22.1 (K): now also J19F2.2
- net at D78.1 (K): now also J26F1.2
- net at D23.1 (K): now also J19G1.2
- net at D79.1 (K): now also J26G1.2
- net at D24.1 (K): now also J19H1.2
- net at D80.1 (K): now also J26H1.2
- net at D76.1 (K), SW9.2: now also J26D1.2
- net at D75.1 (K), SW8.2: now also J26C1.2
- net at D74.1 (K), SW7.2: now also J26B1.2
- net at D73.1 (K), SW6.2: now also J26A1.2
- net at D17.1 (K), SW1.2: now also J19C2.2
- net at D18.1 (K), SW2.2: now also J19B1.2
- net at D19.1 (K), SW3.2: now also J19C1.2
- net at D20.1 (K), SW4.2: now also J19D1.2
- net at D21.1 (K), SW5.2: now also J19F1.2
