File: Prototype PCBs/Shield v.2/Shield v.2.sch (KiCad schematic (older format))
At the start: 81 parts, among them J1 Conn_01x04, J10 i2cA, J11 i2cB, J14 Conn_SysBut, J15 Conn_bLight, J16 Conn_SysLED, J17 LEDs_A, J18 LEDs_B, J2 Conn_01x06, J3 Conn_01x04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

Commit message: Corrected Unavailable 74HC4051 footprint on Shield Board
Parts:
- U1: footprint Package_SO:SSOP-16_3.9x4.9mm_P0.635mm -> Package_SO:TSSOP-16_4.4x5mm_P0.65mm
Changed lines of the file:
@@
 F 0 "U1" H 1250 4878 50  0000 C CNN
 F 1 "74HC4051" H 1250 4787 50  0000 C CNN
-F 2 "Package_SO:SSOP-16_3.9x4.9mm_P0.635mm" H 1200 3800 50  0001 C CNN
+F 2 "Package_SO:TSSOP-16_4.4x5mm_P0.65mm" H 1200 3800 50  0001 C CNN
 F 3 "http://www.ti.com/lit/ds/symlink/cd74hc4051.pdf" H 1200 3800 50  0001 C CNN
 	1    1200 4200
